File: pcb/Produzierte_Platinen/megashield_svn_1.2_geschlossen/ardumower mega shield svn.sch (KiCad schematic (older format))
At the start: 189 parts, among them K3 RELAY_2RT, P1 Sonar C, P10 GPS, P11 Bumper, P12 P.Left, P13 RC Remote, P14 Meas V, P15 Left, P16 V.OUT, P17 V.OUT, P18 Right, P19 Tilt sens, P2 Sonar R, P20 Button, P21 DropRight, P22 Res.AD6, P23 I2C Res.1, P24 I2C Res.2, P25 Res.Pin9, P26 Res.Pin4, P27 Res.Pin0, P28 Res.Pin8, P29 Res.Pin1, P3 Sonar L, P30 P.Right, P31 DropLeft, P32 Voltage header GND, P33 Voltage header 5V, P34 Voltage header 3,3V, P35 Resv.Pin49, P36 Res24V-2, P37 Mower, P38 Status LEDs GND, P39 Res24V-1, P4 MowRpm, P40 UserSwitsch, P41 Rain, P42 Charger connector, P43 Battery, P44 Wlan, P45 I2C Res.3, P46 I2C Res.4, P5 IMU Compas, P6 Lawn sens, P7 Status LEDs, P8 ODO Right, P9 ODO Left, Q1 BC547, U1 DC 10V, U10 I2C_5-3V, U11 Wlan_ESP8266, U2 Bluetooth_CZ_HC_05, U3 INA169, U4 LM350T, U5 INA169, U6 DC 3,3V, U7 DC 5V, U8 DS1307+, U9 Wlan_ESP8266

Commit message: Typo...
Other:
- note added: "LED Anzeigen - Hardware:\n\nLed 3V grün - Betriebsanzeige Versorgungsspannung\nLED 24V grün - Betriebsanzeige Versorgungsspannung R2 für 12V anpassen\nLED 5V grün - Betriebsanzeige Versorgungsspannung\nLED Station - gelb - Statusanzeige ob Mover in Ladestation\n\n----------------------------------------------------------\n\nLED Anzeigen - Software:\n\nDual LED z.B:\nDual LED grün Dauerlicht - Mov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"
- note removed: "LED Anzeigen - Hardware:\n\nLed 3V grün - Betriebsanzeige Versorgungsspannung\nLED 24V grün - Betriebsanzeige Versorgungsspannung R2 für 12 V anpassen\nLED 5V grün - Betriebsanzeige Versorgungsspannung\nLED Station - gelb - Statusanzeige ob Mover in Ladestation\n\n----------------------------------------------------------\n\nLED Anzeigen - Software:\n\nDual LED z.B:\nDual LED grün. Dauerlicht - M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"
Changed lines of the file:
@@
 $EndComp
 Text Notes 8700 -225 0    60   ~ 0
-LED Anzeigen - Hardware:\n\nLed 3V grün -   Betriebsanzeige Versorgungsspannung\nLED 24V grün - Betriebsanzeige Versorgungsspannung R2 für 12 V anpassen\nLED 5V grün -   Betriebsanzeige Versorgungsspannung\nLED Station - gelb - Statusanzeige ob Mover in Ladestation\n\n----------------------------------------------------------\n\nLED Anzeigen - Software:\n\nDual LED z.B:\nDual LED grün. Dauerlicht - Mover innerhalb Perimeter\nDual LED grün+rot = Orange - Dauerlicht Mover außerhalb Perimeter\nDual LED grün+rot = Orange - Blinkt Mover findet  Perimeter nicht oder sucht danach\nDual LED rot =  Blinkt Fehler kurzseitig Überlast Antriebmotor Treibe oder Mähmotor. \nDual LED rot - Dauerlicht - Fehler muß für weiterfahren durch drücken \nvon Button zurückgesetzt werden\n----------------------------------------------------------\n\nLED Status - grün Dauerlicht - warte auf Eingabe\n\nLED Status - grün blinken 1 bis 5 mal hintereinander\nmit länger Pause dazwischen für Anzeige in welchen\nBetriebsmodi sich der Mover befindet
+LED Anzeigen - Hardware:\n\nLed 3V grün -   Betriebsanzeige Versorgungsspannung\nLED 24V grün - Betriebsanzeige Versorgungsspannung R2 für 12V anpassen\nLED 5V grün -   Betriebsanzeige Versorgungsspannung\nLED Station - gelb - Statusanzeige ob Mover in Ladestation\n\n----------------------------------------------------------\n\nLED Anzeigen - Software:\n\nDual LED z.B:\nDual LED grün Dauerlicht - Mover innerhalb Perimeter\nDual LED grün+rot = Orange - Dauerlicht Mower außerhalb Perimeter\nDual LED grün+rot = Orange - Blinkt > Mower findet Perimeter nicht oder sucht danach\nDual LED rot =  Blinkt > Fehler kurzzeitig Überlast Antriebmotor Treiber oder Mähmotor. \nDual LED rot - Dauerlicht - Fehler muss für weiterfahren durch drücken \nvon Button zurückgesetzt werden\n----------------------------------------------------------\n\nLED Status - grün Dauerlicht - warte auf Eingabe\n\nLED Status - grün blinken 1 bis 5 mal hintereinander\nmit länger Pause dazwischen für Anzeige in welchem\nBetriebsmodi sich der Mower befindet
 $Comp
 L JUMPER JP3
